File: pcb/v2/kolsch.kicad_pcb (KiCad board)
At the start: 4 copper layers, 90 x 50 mm, 211 parts, among them J1 TYPE-C-31-M-12-FIXED, J2 USB_A_Stacked, J3 AudioJack4, J4 MICROSD, SW1 BOOT, U1 CCGM1A1, U10 TLV62569DDC, U11 TLV62569DDC, U2 W989D6DBGX6, U3 LSF0108PWR, U4 RP2040, U5 AT25FF321A-SSHN-B, U6 48MHz, U7 NCP164ASN180T1G, U8 LSF0108PWR, U9 TLV62569DDC, Y1 ECS-80-12-33-JGN-TR-12MHZ

Commit message: update schematics
Parts:
- C84: value 10nF -> 100nF
- R73: value 1R -> 22R
